Commit message: aubo_i5 add gripper urdf, add easy_handeye

File: aubo_ros_meta/src/aubo_meta/aubo_description/urdf/aubo_i5.urdf (robot description, URDF)
Before this commit: robot aubo_i5, 10 links, 9 joints
Links:
- added link camera_base, mass 0; collision box size=0.15 0.05 0.005; visual box size=0.15 0.05 0.005
- added link camera_link; collision box size=0.05 0.05 0.05; visual box size=0.05 0.05 0.05
- link gripper_Link: geometry collision cylinder length=0.20 radius=0.03; visual cylinder length=0.20 radius=0.05
Joints:
- added joint camera_base_joint: type fixed, parent wrist3_Link, child camera_base, origin xyz=0 0 0 rpy=0 0 0
- added joint camera_joint: type fixed, parent camera_base, child camera_link, origin xyz=0 0 0.0 rpy=0 0 0
- joint gripper_joint: parent wrist3_Link -> camera_base

File: aubo_ros_meta/src/aubo_meta/aubo_description/urdf/aubo_i5.urdf.xacro (robot description, xacro)
@@ -204,5 +204,6 @@
         <limit lower="-3.04" upper="3.04" effort="0" velocity="0" />
     </joint>
-    <link name="gripper_Link">
+    <!--/////////////////////////////// camera_base ////////////////////////////////////-->
+    <link name="camera_base">
         <inertial>
             <origin xyz="0 0 0" rpy="0 0 0" />
@@ -211,32 +212,87 @@
         </inertial>
         <visual>
-            <origin xyz="0 0 0.1" rpy="0 0 0" />
+            <origin xyz="0.055 0 0.0025" rpy="0 0 0" />
+            <geometry>
+                <box size="0.15 0.05 0.005" />
+            </geometry>
+            <material name="">
+                <color rgba="1 1 1 1" />
+            </material>
+        </visual>
+        <collision>
+            <origin xyz="0.055 0 0.0025" rpy="0 0 0" />
+            <geometry>
+                <box size="0.15 0.05 0.005" />
+            </geometry>
+        </collision>
+    </link>
+    <!--/////////////////////////////// camera_base_joint ////////////////////////////////////-->
+    <joint name="camera_base_joint" type="fixed">
+        <origin xyz="0 0 0" rpy="0 0 0" />
+        <parent link="wrist3_Link" />
+        <child link="camera_base" />
+    </joint>
+    <!--/////////////////////////////// gripper_Link ////////////////////////////////////-->
+    <link name="gripper_Link">
+        <inertial>
+            <origin xyz="0 0 0" rpy="0 0 0" />
+            <mass value="0" />
+            <inertia ixx="0" ixy="0" ixz="0" iyy="0" iyz="0" izz="0" />
+        </inertial>
+        <visual>
+            <origin xyz="0 0 0.105" rpy="0 0 0" />
             <geometry>
                 <!-- <mesh filename="package://aubo_description/meshes/aubo_i5/visual/wrist3_Link.DAE" /> -->
-                <cylinder radius="0.03" length="0.20"/>
-            </geometry>
-            <material name="">
-                <color rgba="1 1 1 1" />
-            </material>
-        </visual>
-        <collision>
-            <origin xyz="0 0 0.1" rpy="0 0 0" />
+                <cylinder radius="0.05" length="0.20" />
+            </geometry>
+            <material name="">
+                <color rgba="1 1 1 1" />
+            </material>
+        </visual>
+        <collision>
+            <origin xyz="0 0 0.105" rpy="0 0 0" />
             <geometry>
                 <!-- <mesh filename="package://aubo_description/meshes/aubo_i5/collision/wrist3_Link.STL" /> -->
-                <cylinder radius="0.03" length="0.20"/>
-            </geometry>
-        </collision>
-    </link>
+                <cylinder radius="0.03" length="0.20" />
+            </geometry>
+        </collision>
+    </link>
+    <!--/////////////////////////////// gripper_joint ////////////////////////////////////-->
     <joint name="gripper_joint" type="fixed">
         <origin xyz="0 0 0" rpy="0 0 0" />
-        <parent link="wrist3_Link" />
+        <parent link="camera_base" />
         <child link="gripper_Link" />
     </joint>
-    <link name="gripper_tip_Link">
-    </link>
+    <!--/////////////////////////////// gripper_tip_Link ////////////////////////////////////-->
+    <link name="gripper_tip_Link"></link>
+    <!--/////////////////////////////// gripper_tip_joint ////////////////////////////////////-->
     <joint name="gripper_tip_joint" type="fixed">
         <origin xyz="0 0 0.2" rpy="0 0 0" />
         <parent link="gripper_Link" />
         <child link="gripper_tip_Link" />
+    </joint>
+    <!--/////////////////////////////// camera_link ////////////////////////////////////-->
+    <link name="camera_link">
+        <visual>
+            <origin xyz="0.105 0 0.03" rpy="0 0 0" />
+            <geometry>
+                <box size="0.05 0.05 0.05" />
+            </geometry>
+            <material name="">
+                <color rgba="1 1 1 1" />
+            </material>
+        </visual>
+        <collision>
+            <origin xyz="0.105 0 0.03" rpy="0 0 0" />
+            <geometry>
+                <box size="0.05 0.05 0.05" />
+            </geometry>
+        </collision>
+    </link>
+    <!--/////////////////////////////// camera_joint ////////////////////////////////////-->
+    <joint name="camera_joint" type="fixed">
+        <origin xyz="0 0 0.0" rpy="0 0 0" />
+        <parent link="camera_base" />
+        <child link="camera_link" />
     </joint>
     <link name="world" />

File: aubo_ros_meta/src/aubo_meta/aubo_gazebo/urdf/aubo_i5.xacro (robot description, xacro)
@@ -247,6 +247,6 @@
         <limit lower="-3.04" upper="3.04" effort="300" velocity="100" />
     </joint>
-    <!-- ////////////////////////////////// i5 gripper_link /////////////////////////////////////////// -->
-    <link name="gripper_Link">
+    <!--/////////////////////////////// camera_base ////////////////////////////////////-->
+    <link name="camera_base">
         <inertial>
             <origin xyz="0 0 0" rpy="0 0 0" />
@@ -255,15 +255,44 @@
         </inertial>
         <visual>
-            <origin xyz="0 0 0.1" rpy="0 0 0" />
+            <origin xyz="0.055 0 0.0025" rpy="0 0 0" />
+            <geometry>
+                <box size="0.15 0.05 0.005" />
+            </geometry>
+            <material name="">
+                <color rgba="1 1 1 1" />
+            </material>
+        </visual>
+        <collision>
+            <origin xyz="0.055 0 0.0025" rpy="0 0 0" />
+            <geometry>
+                <box size="0.15 0.05 0.005" />
+            </geometry>
+        </collision>
+    </link>
+    <!--/////////////////////////////// camera_base_joint ////////////////////////////////////-->
+    <joint name="camera_base_joint" type="fixed">
+        <origin xyz="0 0 0" rpy="0 0 0" />
+        <parent link="wrist3_Link" />
+        <child link="camera_base" />
+    </joint>
+    <!--/////////////////////////////// gripper_Link ////////////////////////////////////-->
+    <link name="gripper_Link">
+        <inertial>
+            <origin xyz="0 0 0" rpy="0 0 0" />
+            <mass value="0" />
+            <inertia ixx="0" ixy="0" ixz="0" iyy="0" iyz="0" izz="0" />
+        </inertial>
+        <visual>
+            <origin xyz="0 0 0.105" rpy="0 0 0" />
             <geometry>
                 <!-- <mesh filename="package://aubo_description/meshes/aubo_i5/visual/wrist3_Link.DAE" /> -->
-                <cylinder radius="0.03" length="0.20" />
-            </geometry>
-            <material name="">
-                <color rgba="1 1 1 1" />
-            </material>
-        </visual>
-        <collision>
-            <origin xyz="0 0 0.1" rpy="0 0 0" />
+                <cylinder radius="0.05" length="0.20" />
+            </geometry>
+            <material name="">
+                <color rgba="1 1 1 1" />
+            </material>
+        </visual>
+        <collision>
+            <origin xyz="0 0 0.105" rpy="0 0 0" />
             <geometry>
                 <!-- <mesh filename="package://aubo_description/meshes/aubo_i5/collision/wrist3_Link.STL" /> -->
@@ -272,15 +301,41 @@
         </collision>
     </link>
+    <!--/////////////////////////////// gripper_joint ////////////////////////////////////-->
     <joint name="gripper_joint" type="fixed">
         <origin xyz="0 0 0" rpy="0 0 0" />
-        <parent link="wrist3_Link" />
+        <parent link="camera_base" />
         <child link="gripper_Link" />
     </joint>
-    <!-- ////////////////////////////////// i5 gripper_tip_link /////////////////////////////////////////// -->
+    <!--/////////////////////////////// gripper_tip_Link ////////////////////////////////////-->
     <link name="gripper_tip_Link"></link>
+    <!--/////////////////////////////// gripper_tip_joint ////////////////////////////////////-->
     <joint name="gripper_tip_joint" type="fixed">
         <origin xyz="0 0 0.2" rpy="0 0 0" />
         <parent link="gripper_Link" />
         <child link="gripper_tip_Link" />
+    </joint>
+    <!--/////////////////////////////// camera_link ////////////////////////////////////-->
+    <link name="camera_link">
+        <visual>
+            <origin xyz="0.105 0 0.03" rpy="0 0 0" />
+            <geometry>
+                <box size="0.05 0.05 0.05" />
+            </geometry>
+            <material name="">
+                <color rgba="1 1 1 1" />
+            </material>
+        </visual>
+        <collision>
+            <origin xyz="0.105 0 0.03" rpy="0 0 0" />
+            <geometry>
+                <box size="0.05 0.05 0.05" />
+            </geometry>
+        </collision>
+    </link>
+    <!--/////////////////////////////// camera_joint ////////////////////////////////////-->
+    <joint name="camera_joint" type="fixed">
+        <origin xyz="0 0 0.0" rpy="0 0 0" />
+        <parent link="camera_base" />
+        <child link="camera_link" />
     </joint>
     <!-- /////////////////////////////////   i5 pedestal_Link   ////////////////////////////////////// -->
