Commit message: moveit add octpmap

File: aubo_ros_meta/src/aubo_meta/aubo_description/urdf/aubo_i5.urdf.xacro (robot description, xacro)
@@ -302,3 +302,25 @@
         <origin xyz="0.0 0.0 0.0" rpy="0.0 0.0 0.0" />
     </joint>
+    <!-- <link name="cam_eyetohand">
+        <visual>
+            <origin xyz="-0.863 -0.410 0.721" rpy="-1.6257138 0.0310401 -0.6831306" />
+            <geometry>
+                <box size="0.05 0.05 0.05" />
+            </geometry>
+            <material name="">
+                <color rgba="1 1 1 1" />
+            </material>
+        </visual>
+        <collision>
+            <origin xyz="-0.863 -0.410 0.721" rpy="-1.6257138 0.0310401 -0.6831306" />
+            <geometry>
+                <box size="0.05 0.05 0.05" />
+            </geometry>
+        </collision>
+    </link>
+    <joint name="cam_eyetohand_joint" type="fixed">
+        <origin xyz="-0.863 -0.410 0.721" rpy="-1.6257138 0.0310401 -0.6831306" />
+        <parent link="base_link" />
+        <child link="cam_eyetohand" />
+    </joint> -->
 </robot>

File: aubo_ros_meta/src/aubo_meta/aubo_gazebo/urdf/aubo_i5.xacro (robot description, xacro)
@@ -354,4 +354,8 @@
     <!-- /////////////////////////////////   world   ////////////////////////////////////// -->
     <link name="world" />
+    <!-- /////////////////////////////////   gazebo color   ////////////////////////////////////// -->
+    <gazebo reference="pedestal_Link">
+        <material>Gazebo/Grey</material>
+    </gazebo>
     <joint name="world_joint" type="fixed">
         <parent link="world" />
@@ -359,8 +363,4 @@
         <origin xyz="0.0 0.0 0.1" rpy="0.0 0.0 0.0" />
     </joint>
-    <!-- /////////////////////////////////   gazebo color   ////////////////////////////////////// -->
-    <gazebo reference="pedestal_Link">
-        <material>Gazebo/Grey</material>
-    </gazebo>
     <!--////////////////////////////////// Transmissions for ROS Control //////////////////////////-->
     <xacro:macro name="aubo_arm_transmission" params="joint_name">
@@ -388,3 +388,25 @@
         </plugin>
     </gazebo>
+    <!-- <link name="cam_eyetohand">
+        <visual>
+            <origin xyz="0 0 0" rpy="0 0 0" />
+            <geometry>
+                <box size="0.05 0.05 0.05" />
+            </geometry>
+            <material name="">
+                <color rgba="1 1 1 1" />
+            </material>
+        </visual>
+        <collision>
+            <origin xyz="0 0 0" rpy="0 0 0" />
+            <geometry>
+                <box size="0.05 0.05 0.05" />
+            </geometry>
+        </collision>
+    </link> -->
+    <!-- <joint name="cam_eyetohand_joint" type="fixed">
+        <origin xyz="-0.863 -0.410 0.721" rpy="-1.6257138 0.0310401 -0.6831306" />
+        <parent link="base_link" />
+        <child link="cam_eyetohand" />
+    </joint> -->
 </robot>
